File: layouts/default/default.kicad_pcb (KiCad board)
At the start: 2 copper layers, 49 parts

Commit message: Add USB-C connector, boot and reset buttons to ESP32-C6 driver
Add programming interface: USB-C (TYPE-C-31-M-12) with CC pull-downs,
boot button (GPIO9→GND) and reset button (EN→GND) using XKB tactile
switches. Remove redundant USB ElectricLogic definitions.

Co-Authored-By: Claude Opus 4.6 <noreply@anthropic.com>
Parts:
- added R18: 5100Ω, UNI_ROYAL_0402WGF5101TCE:R0402, F.Cu at (30.0, -10.0)
- added R19: 5100Ω, UNI_ROYAL_0402WGF5101TCE:R0402, F.Cu at (30.0, 0.00)
- added SW1: , XKB_Connectivity_TS_1187A_B_A_B:SW-SMD_4P-L5.1-W5.1-P3.70-LS6.5-TL_H1.5, F.Cu at (0.00, 0.00)
- added SW2: , XKB_Connectivity_TS_1187A_B_A_B:SW-SMD_4P-L5.1-W5.1-P3.70-LS6.5-TL_H1.5, F.Cu at (10.0, 0.00)
- added USBC1: , Korean_Hroparts_Elec_TYPE_C_31_M_12:USB-C_SMD-TYPE-C-31-M-12_1, F.Cu at (20.0, 0.00)
Connections:
- net 23 renamed A

Commit message: Route 4-layer PCB with corrected component placement
Rewrote placement based on actual netlist assignments (atopile ref
designators differ from schematic expectations). 60x48mm board with
4-layer stackup, GND zones on In1.Cu/F.Cu/B.Cu. Autorouted with
KiCadRoutingTools: 24/25 signal nets routed, 99/99 multipoint pads,
81 vias. One minor SDA disconnection on U1.8 remains.

Co-Authored-By: Claude Opus 4.6 <noreply@anthropic.com>
Parts:
- R14, R15, R2, R3: moved to B.Cu
- moved R11 385.0 mm to (125.0, 115.0)
- moved R9 371.0 mm to (122.0, 111.0)
- moved R6 366.1 mm to (129.0, 116.0)
- moved C9 336.1 mm to (112.0, 116.0)
- moved C7 309.0 mm to (125.0, 109.0), turned to 90 degrees
- moved C3 296.3 mm to (133.0, 116.0)
- moved R10 243.0 mm to (122.0, 113.0)
- moved C5 235.3 mm to (108.0, 115.0)
- moved R7 222.3 mm to (108.0, 112.0)
- moved R5 204.2 mm to (129.0, 114.0)
- moved C6 187.8 mm to (103.0, 107.0), turned to 90 degrees
- moved C14 187.4 mm to (143.0, 92.0), turned to 90 degrees
- moved CN1 184.9 mm to (148.0, 123.0)
- moved U6 178.2 mm to (152.0, 93.0)
- moved R17 176.2 mm to (146.0, 92.0), turned to 90 degrees
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Routing:
- net hv: track 0.00 -> 121.6 mm, vias 0 -> 19
- net Vbatr-hv: track 0.00 -> 80.8 mm, vias 0 -> 13
- net SDA: track 3.87 -> 57.0 mm, vias 0 -> 2
- net SCL: track 3.92 -> 48.8 mm, vias 0 -> 10
- net c_en-power-hv: track 0.00 -> 44.2 mm, vias 0 -> 4
- net A: track 0.00 -> 42.3 mm, vias 0 -> 3
- net 18: track 0.00 -> 29.0 mm, vias 0 -> 4
- net Coutsns-power-hv: track 0.00 -> 27.4 mm, vias 0 -> 4
- net anode: track 0.00 -> 26.1 mm
- net 0: track 24.9 -> 0.00 mm, vias 8 -> 0
- net 17: track 0.00 -> 23.6 mm, vias 0 -> 4
- net 1: track 0.00 -> 22.3 mm
- net Vpvr-hv: track 0.00 -> 18.4 mm
- net Cout1-power-hv: track 0.00 -> 18.0 mm, vias 0 -> 4
- net cathode: track 0.00 -> 17.1 mm, vias 0 -> 3
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- added copper zone on B.Cu, net lv
- added copper zone on F.Cu, net lv
- added copper zone on In1.Cu, net lv
Other:
- board outline added: 60 x 48 mm
- copper layers 2 -> 4
