File: quilter_upload/default.kicad_pcb (KiCad board)
At the start: 4 copper layers, 60 x 48 mm, 54 parts

Commit message: Add schematic generation, Quilter prep scripts, and updated PCB
- Add generate_schematic.py to create KiCad 9 schematic from design
- Add prepare_for_quilter.py to strip and prepare PCB for Quilter AI routing
- Add generated schematic (default.kicad_sch)
- Add quilter_upload/ directory with prepared KiCad project files
- Update PCB layout with KiCad 9 formatting changes

Co-Authored-By: Claude Opus 4.6 <noreply@anthropic.com>
Parts:
- moved USBC1 265.3 mm to (165.0, 343.0)
- moved SW2 248.2 mm to (165.0, 333.0)
- moved C13 232.1 mm to (165.0, 318.0)
- moved C11 228.6 mm to (165.0, 338.0)
- moved U3 221.7 mm to (165.0, 328.0)
- moved R4 210.2 mm to (165.0, 323.0)
- moved R10 204.6 mm to (165.0, 313.0)
- moved R16 202.5 mm to (165.0, 288.0)
- moved R5 197.3 mm to (165.0, 308.0)
- moved R13 194.0 mm to (165.0, 298.0)
- moved R17 187.0 mm to (165.0, 278.0)
- moved CN1 180.8 mm to (165.0, 303.0)
- moved LED1 180.0 mm to (165.0, 293.0)
- moved C5 177.4 mm to (165.0, 283.0)
- moved C16 174.2 mm to (165.0, 263.0)
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Routing:
- net hv: track 121.6 -> 0.00 mm, vias 19 -> 0
- net Vbatr-hv: track 80.8 -> 0.00 mm, vias 13 -> 0
- net SDA: track 57.0 -> 0.00 mm, vias 2 -> 0
- net SCL: track 48.8 -> 0.00 mm, vias 10 -> 0
- net c_en-power-hv: track 44.2 -> 0.00 mm, vias 4 -> 0
- net A: track 42.3 -> 0.00 mm, vias 3 -> 0
- net 18: track 29.0 -> 0.00 mm, vias 4 -> 0
- net Coutsns-power-hv: track 27.4 -> 0.00 mm, vias 4 -> 0
- net anode: track 26.1 -> 0.00 mm
- net 17: track 23.6 -> 0.00 mm, vias 4 -> 0
- net 1: track 22.3 -> 0.00 mm
- net Vpvr-hv: track 18.4 -> 0.00 mm
- net Cout1-power-hv: track 18.0 -> 0.00 mm, vias 4 -> 0
- net cathode: track 17.1 -> 0.00 mm, vias 3 -> 0
- net Cinsns-power-hv: track 15.3 -> 0.00 mm, vias 2 -> 0
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- removed copper zone on B.Cu, net lv
- removed copper zone on F.Cu, net lv
- removed copper zone on In1.Cu, net lv
Other:
- board size 60 x 48 mm -> 45 x 38 mm
- copper layers 4 -> 2

Commit message: Add OpenSCAD enclosure, STEP exports, PCB previews, and Quilter candidates
- Add OpenSCAD parametric enclosure (enclosure.scad) with full assembly exports
- Add STEP export pipeline (export_all.py) with assembly components
- Add STL/STEP files for base, lid, ball/nut/socket hardware
- Add 3MF print files for hardware parts
- Add PCB preview PDF/SVG for default layout
- Add Quilter 4-layer and 6-layer PCB candidates
- Add setup_board.py for board setup automation
- Update enclosure.py and view_enclosure.py (build123d)
- Update main.ato and micromppt.ato (circuit refinements)
- Update prepare_for_quilter.py and ato.yaml
- Add docs/power_budget.md

Co-Authored-By: Claude Sonnet 4.6 <noreply@anthropic.com>
Parts:
- removed CN2: , JST_Sales_America_B2B_PH_K_S_LF__SN:CONN-TH_B2B-PH-K-S
- removed D2: Vf ℝ+V, GOODWORK_B5819W:SOD-123F_L2.7-W1.6-LS3.8-RD-1
- removed F1: , Littelfuse_0603L150SLYR:F0603
- added H1: , MountingHole_3_2_M3:MountingHole_3.2_M3, F.Cu at (103.5, 81.5)
- added H2: , MountingHole_3_2_M3:MountingHole_3.2_M3, F.Cu at (156.5, 81.5)
- added H3: , MountingHole_3_2_M3:MountingHole_3.2_M3, F.Cu at (103.5, 122.5)
- added H4: , MountingHole_3_2_M3:MountingHole_3.2_M3, F.Cu at (156.5, 122.5)
- R14, R15, R2, R3: moved to F.Cu
- moved USBC1 258.1 mm to (105.0, 92.0), turned to -90 degrees
- moved SW2 227.1 mm to (105.0, 114.0)
- moved CN1 184.4 mm to (130.0, 122.0), turned to 180 degrees
- moved R15 180.6 mm to (180.0, 273.0), turned to 0 degrees
- moved CN4 161.8 mm to (156.0, 91.5), turned to -90 degrees
- moved U5 118.3 mm to (130.0, 85.0)
- moved CN5 96.4 mm to (156.0, 112.0), turned to -90 degrees
- moved R14 86.3 mm to (180.0, 173.0), turned to 0 degrees
- moved R2 86.3 mm to (180.0, 168.0)
- moved R3 76.5 mm to (180.0, 153.0)
- moved SW1 71.6 mm to (105.0, 104.0)
- moved CN3 58.8 mm to (115.0, 122.0), turned to 180 degrees
- moved C11 52.2 mm to (180.0, 288.0), turned to 180 degrees
- moved C13 52.2 mm to (180.0, 268.0)
- moved R10 52.2 mm to (180.0, 263.0)
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Connections:
- net cathode renamed Vbatr-lv
Other:
- board size 45 x 38 mm -> 60 x 48 mm
- copper layers 2 -> 4
- board text added: "BATT"
- board text added: "BOOT"
- board text added: "EC"
- board text added: "RESET"
- board text added: "SOIL"
- board text added: "SOLAR"
- board text added: "USB"
